File: Pico2WKeyboard.kicad_sch (KiCad schematic)
At the start: 72 parts, among them SW1 SW_Push, SW10 SW_Push, SW11 SW_Push, SW12 SW_Push, SW13 SW_Push, SW14 SW_Push, SW15 SW_Push, SW16 SW_Push, SW17 SW_Push, SW18 SW_Push, SW19 SW_Push, SW2 SW_Push, SW20 SW_Push, SW21 SW_Push, SW22 SW_Push, SW23 SW_Push, SW24 SW_Push, SW25 SW_Push, SW3 SW_Push, SW4 SW_Push, SW5 SW_Push, SW6 SW_Push, SW7 SW_Push, SW8 SW_Push, SW9 SW_Push, U1 24C16N

Commit message: Added LCSC numbers
Parts:
- A1: LCSC (none) -> C42394205
- C1: LCSC (none) -> C1525
- D1, D10, D11, D12, D13, D14, D15, D16, D17, D18, D19, D2, D20, D21, D22, D23, D24, D25, D3, D4, D5, D6, D7, D8, D9: LCSC (none) -> C402212
- D26: LCSC (none) -> C389522
- D27, D28, D29: LCSC (none) -> C2286
- R1, R10, R11, R2, R3, R4, R9: LCSC (none) -> C25804
- R5, R6, R7, R8: LCSC (none) -> C23138
- SW1, SW10, SW11, SW12, SW13, SW14, SW15, SW16, SW17, SW18, SW19, SW2, SW20, SW21, SW22, SW23, SW24, SW25, SW3, SW4, SW5, SW6, SW7, SW8, SW9: LCSC (none) -> C393938
- U1: LCSC (none) -> C18723551
